Commit message: Update : update cartrasche urdf

File: src/cartrasche/cartrasche_description/urdf/cartrasche.xacro (robot description, xacro)
@@ -6,7 +6,7 @@
 <link name="base_link">
   <inertial>
-    <origin xyz="-0.17500000000000093 0.1465379545676244 -0.04167420563757363" rpy="0 0 0"/>
-    <mass value="14.854275644982799"/>
-    <inertia ixx="0.311009" iyy="0.269977" izz="0.551767" ixy="0.0" iyz="0.004993" ixz="-0.0"/>
+    <origin xyz="-8.899261942654923e-16 0.11274549780959403 0.062447509482163" rpy="0 0 0"/>
+    <mass value="23.746934326209"/>
+    <inertia ixx="0.59366" iyy="0.36641" izz="0.768564" ixy="0.0" iyz="0.088771" ixz="-0.0"/>
   </inertial>
   <visual>
@@ -24,55 +24,106 @@
   </collision>
 </link>
-<link name="Wheel_L_1">
+<link name="wheelL_1">
   <inertial>
-    <origin xyz="-0.004962223004344377 3.726186026398182e-15 6.522560269672795e-16" rpy="0 0 0"/>
+    <origin xyz="-0.004962223004344346 4.211908599671688e-15 5.4392540028557067e-17" rpy="0 0 0"/>
+    <mass value="3.060084322980661"/>
+    <inertia ixx="0.004797" iyy="0.0028" izz="0.0028" ixy="0.0" iyz="0.0" ixz="-0.0"/>
+  </inertial>
+  <visual>
+    <origin xyz="-0.207 -0.06 -0.0" rpy="0 0 0"/>
+    <geometry>
+      <mesh filename="package://cartrasche_description/meshes/wheelL_1.stl" scale="0.001 0.001 0.001"/>
+    </geometry>
+    <material name="silver"/>
+  </visual>
+  <collision>
+    <origin xyz="-0.207 -0.06 -0.0" rpy="0 0 0"/>
+    <geometry>
+      <mesh filename="package://cartrasche_description/meshes/wheelL_1.stl" scale="0.001 0.001 0.001"/>
+    </geometry>
+  </collision>
+</link>
+<link name="wheelR_1">
+  <inertial>
+    <origin xyz="0.004962223004344346 -4.198030811863873e-15 5.4392540028557067e-17" rpy="0 0 0"/>
     <mass value="3.060084322980661"/>
     <inertia ixx="0.004797" iyy="0.0028" izz="0.0028" ixy="0.0" iyz="0.0" ixz="0.0"/>
   </inertial>
   <visual>
-    <origin xyz="-0.032 -0.06 0.063" rpy="0 0 0"/>
+    <origin xyz="0.207 -0.06 -0.0" rpy="0 0 0"/>
     <geometry>
-      <mesh filename="package://cartrasche_description/meshes/Wheel_L_1.stl" scale="0.001 0.001 0.001"/>
+      <mesh filename="package://cartrasche_description/meshes/wheelR_1.stl" scale="0.001 0.001 0.001"/>
     </geometry>
     <material name="silver"/>
   </visual>
   <collision>
-    <origin xyz="-0.032 -0.06 0.063" rpy="0 0 0"/>
+    <origin xyz="0.207 -0.06 -0.0" rpy="0 0 0"/>
     <geometry>
-      <mesh filename="package://cartrasche_description/meshes/Wheel_L_1.stl" scale="0.001 0.001 0.001"/>
+      <mesh filename="package://cartrasche_description/meshes/wheelR_1.stl" scale="0.001 0.001 0.001"/>
     </geometry>
   </collision>
 </link>
-<link name="Wheel_R_1">
+<link name="ridar_1">
   <inertial>
-    <origin xyz="0.004962223004343791 -4.198030811863873e-15 1.3877787807814457e-17" rpy="0 0 0"/>
-    <mass value="3.060084322980661"/>
-    <inertia ixx="0.004797" iyy="0.0028" izz="0.0028" ixy="0.0" iyz="-0.0" ixz="0.0"/>
+    <origin xyz="-7.385233546074017e-18 -2.7755575615628914e-17 0.010000000000000009" rpy="0 0 0"/>
+    <mass value="0.6042068071016568"/>
+    <inertia ixx="0.000205" iyy="0.000205" izz="0.00037" ixy="-0.0" iyz="0.0" ixz="-0.0"/>
   </inertial>
   <visual>
-    <origin xyz="0.382 -0.06 0.063" rpy="0 0 0"/>
+    <origin xyz="-0.0 -0.075 -0.193" rpy="0 0 0"/>
     <geometry>
-      <mesh filename="package://cartrasche_description/meshes/Wheel_R_1.stl" scale="0.001 0.001 0.001"/>
+      <mesh filename="package://cartrasche_description/meshes/ridar_1.stl" scale="0.001 0.001 0.001"/>
     </geometry>
     <material name="silver"/>
   </visual>
   <collision>
-    <origin xyz="0.382 -0.06 0.063" rpy="0 0 0"/>
+    <origin xyz="-0.0 -0.075 -0.193" rpy="0 0 0"/>
     <geometry>
-      <mesh filename="package://cartrasche_description/meshes/Wheel_R_1.stl" scale="0.001 0.001 0.001"/>
+      <mesh filename="package://cartrasche_description/meshes/ridar_1.stl" scale="0.001 0.001 0.001"/>
     </geometry>
   </collision>
 </link>
-<joint name="Rotate1" type="continuous">
-  <origin xyz="0.032 0.06 -0.063" rpy="0 0 0"/>
+<link name="cam_1">
+  <inertial>
+    <origin xyz="0.0 -0.0050000000000000044 0.009999999999999995" rpy="0 0 0"/>
+    <mass value="0.024661502330679874"/>
+    <inertia ixx="1e-06" iyy="1e-06" izz="1e-06" ixy="0.0" iyz="0.0" ixz="-0.0"/>
+  </inertial>
+  <visual>
+    <origin xyz="-0.0 0.02 -0.063" rpy="0 0 0"/>
+    <geometry>
+      <mesh filename="package://cartrasche_description/meshes/cam_1.stl" scale="0.001 0.001 0.001"/>
+    </geometry>
+    <material name="silver"/>
+  </visual>
+  <collision>
+    <origin xyz="-0.0 0.02 -0.063" rpy="0 0 0"/>
+    <geometry>
+      <mesh filename="package://cartrasche_description/meshes/cam_1.stl" scale="0.001 0.001 0.001"/>
+    </geometry>
+  </collision>
+</link>
+<joint name="회전 1" type="continuous">
+  <origin xyz="0.207 0.06 0.0" rpy="0 0 0"/>
   <parent link="base_link"/>
-  <child link="Wheel_L_1"/>
+  <child link="wheelL_1"/>
+  <axis xyz="1.0 -0.0 -0.0"/>
+</joint>
+<joint name="회전 2" type="continuous">
+  <origin xyz="-0.207 0.06 0.0" rpy="0 0 0"/>
+  <parent link="base_link"/>
+  <child link="wheelR_1"/>
   <axis xyz="1.0 0.0 0.0"/>
 </joint>
-<joint name="Rotate2" type="continuous">
-  <origin xyz="-0.382 0.06 -0.063" rpy="0 0 0"/>
+<joint name="회전 3" type="continuous">
+  <origin xyz="0.0 0.075 0.193" rpy="0 0 0"/>
   <parent link="base_link"/>
-  <child link="Wheel_R_1"/>
-  <axis xyz="-1.0 -0.0 0.0"/>
+  <child link="ridar_1"/>
+  <axis xyz="0.0 0.0 1.0"/>
+</joint>
+<joint name="강체 4" type="fixed">
+  <origin xyz="0.0 -0.02 0.063" rpy="0 0 0"/>
+  <parent link="base_link"/>
+  <child link="cam_1"/>
 </joint>
 </robot>
