Commit message: Fix : correct cartrasche_description TF axis

File: cartrasche/cartrasche_description/urdf/cartrasche.xacro (robot description, xacro)
@@ -6,7 +6,7 @@
 <link name="base_link">
   <inertial>
-    <origin xyz="-8.899261942654923e-16 0.11274549780959403 0.062447509482163" rpy="0 0 0"/>
-    <mass value="23.746934326209"/>
-    <inertia ixx="0.59366" iyy="0.36641" izz="0.768564" ixy="0.0" iyz="0.088771" ixz="-0.0"/>
+    <origin xyz="0.0026190663618483622 -2.2185715820021788e-16 0.3388319376922865" rpy="0 0 0"/>
+    <mass value="67.74618432620866"/>
+    <inertia ixx="4.472442" iyy="4.808193" izz="0.950396" ixy="-0.0" iyz="-0.0" ixz="-0.648262"/>
   </inertial>
   <visual>
@@ -26,10 +26,10 @@
 <link name="wheelL_1">
   <inertial>
-    <origin xyz="-0.004962223004344346 4.211908599671688e-15 5.4392540028557067e-17" rpy="0 0 0"/>
+    <origin xyz="-4.260633313594524e-15 -0.0049622230043442905 2.1743594926500883e-17" rpy="0 0 0"/>
     <mass value="3.060084322980661"/>
-    <inertia ixx="0.004797" iyy="0.0028" izz="0.0028" ixy="0.0" iyz="0.0" ixz="-0.0"/>
+    <inertia ixx="0.0028" iyy="0.004797" izz="0.0028" ixy="-0.0" iyz="-0.0" ixz="0.0"/>
   </inertial>
   <visual>
-    <origin xyz="-0.207 -0.06 -0.0" rpy="0 0 0"/>
+    <origin xyz="-0.0 -0.207 -0.0" rpy="0 0 0"/>
     <geometry>
       <mesh filename="package://cartrasche_description/meshes/wheelL_1.stl" scale="0.001 0.001 0.001"/>
@@ -38,5 +38,5 @@
   </visual>
   <collision>
-    <origin xyz="-0.207 -0.06 -0.0" rpy="0 0 0"/>
+    <origin xyz="-0.0 -0.207 -0.0" rpy="0 0 0"/>
     <geometry>
       <mesh filename="package://cartrasche_description/meshes/wheelL_1.stl" scale="0.001 0.001 0.001"/>
@@ -46,10 +46,10 @@
 <link name="wheelR_1">
   <inertial>
-    <origin xyz="0.004962223004344346 -4.198030811863873e-15 5.4392540028557067e-17" rpy="0 0 0"/>
+    <origin xyz="4.347900040796894e-15 0.0049622230043442905 1.0258460747536548e-16" rpy="0 0 0"/>
     <mass value="3.060084322980661"/>
-    <inertia ixx="0.004797" iyy="0.0028" izz="0.0028" ixy="0.0" iyz="0.0" ixz="0.0"/>
+    <inertia ixx="0.0028" iyy="0.004797" izz="0.0028" ixy="-0.0" iyz="-0.0" ixz="0.0"/>
   </inertial>
   <visual>
-    <origin xyz="0.207 -0.06 -0.0" rpy="0 0 0"/>
+    <origin xyz="-0.0 0.207 -0.0" rpy="0 0 0"/>
     <geometry>
       <mesh filename="package://cartrasche_description/meshes/wheelR_1.stl" scale="0.001 0.001 0.001"/>
@@ -58,5 +58,5 @@
   </visual>
   <collision>
-    <origin xyz="0.207 -0.06 -0.0" rpy="0 0 0"/>
+    <origin xyz="-0.0 0.207 -0.0" rpy="0 0 0"/>
     <geometry>
       <mesh filename="package://cartrasche_description/meshes/wheelR_1.stl" scale="0.001 0.001 0.001"/>
@@ -66,10 +66,10 @@
 <link name="ridar_1">
   <inertial>
-    <origin xyz="-7.385233546074017e-18 -2.7755575615628914e-17 0.010000000000000009" rpy="0 0 0"/>
+    <origin xyz="0.0 1.7498924471358617e-16 0.009999999999999898" rpy="0 0 0"/>
     <mass value="0.6042068071016568"/>
-    <inertia ixx="0.000205" iyy="0.000205" izz="0.00037" ixy="-0.0" iyz="0.0" ixz="-0.0"/>
+    <inertia ixx="0.000205" iyy="0.000205" izz="0.00037" ixy="0.0" iyz="-0.0" ixz="-0.0"/>
   </inertial>
   <visual>
-    <origin xyz="-0.0 -0.075 -0.193" rpy="0 0 0"/>
+    <origin xyz="0.015 -0.0 -0.783" rpy="0 0 0"/>
     <geometry>
       <mesh filename="package://cartrasche_description/meshes/ridar_1.stl" scale="0.001 0.001 0.001"/>
@@ -78,5 +78,5 @@
   </visual>
   <collision>
-    <origin xyz="-0.0 -0.075 -0.193" rpy="0 0 0"/>
+    <origin xyz="0.015 -0.0 -0.783" rpy="0 0 0"/>
     <geometry>
       <mesh filename="package://cartrasche_description/meshes/ridar_1.stl" scale="0.001 0.001 0.001"/>
@@ -86,10 +86,10 @@
 <link name="cam_1">
   <inertial>
-    <origin xyz="0.0 -0.0050000000000000044 0.009999999999999995" rpy="0 0 0"/>
+    <origin xyz="0.025000000000000078 -0.07999999999999989 0.009999999999999995" rpy="0 0 0"/>
     <mass value="0.024661502330679874"/>
-    <inertia ixx="1e-06" iyy="1e-06" izz="1e-06" ixy="0.0" iyz="0.0" ixz="-0.0"/>
+    <inertia ixx="1e-06" iyy="1e-06" izz="1e-06" ixy="0.0" iyz="-0.0" ixz="-0.0"/>
   </inertial>
   <visual>
-    <origin xyz="-0.0 0.02 -0.063" rpy="0 0 0"/>
+    <origin xyz="-0.06 -0.08 -0.063" rpy="0 0 0"/>
     <geometry>
       <mesh filename="package://cartrasche_description/meshes/cam_1.stl" scale="0.001 0.001 0.001"/>
@@ -98,5 +98,5 @@
   </visual>
   <collision>
-    <origin xyz="-0.0 0.02 -0.063" rpy="0 0 0"/>
+    <origin xyz="-0.06 -0.08 -0.063" rpy="0 0 0"/>
     <geometry>
       <mesh filename="package://cartrasche_description/meshes/cam_1.stl" scale="0.001 0.001 0.001"/>
@@ -105,23 +105,23 @@
 </link>
 <joint name="회전 1" type="continuous">
-  <origin xyz="0.207 0.06 0.0" rpy="0 0 0"/>
+  <origin xyz="0.0 0.207 0.0" rpy="0 0 0"/>
   <parent link="base_link"/>
   <child link="wheelL_1"/>
-  <axis xyz="1.0 -0.0 -0.0"/>
+  <axis xyz="-0.0 1.0 -0.0"/>
 </joint>
 <joint name="회전 2" type="continuous">
-  <origin xyz="-0.207 0.06 0.0" rpy="0 0 0"/>
+  <origin xyz="0.0 -0.207 0.0" rpy="0 0 0"/>
   <parent link="base_link"/>
   <child link="wheelR_1"/>
-  <axis xyz="1.0 0.0 0.0"/>
+  <axis xyz="-0.0 1.0 -0.0"/>
 </joint>
 <joint name="회전 3" type="continuous">
-  <origin xyz="0.0 0.075 0.193" rpy="0 0 0"/>
+  <origin xyz="-0.015 0.0 0.783" rpy="0 0 0"/>
   <parent link="base_link"/>
   <child link="ridar_1"/>
-  <axis xyz="0.0 0.0 1.0"/>
+  <axis xyz="-0.0 0.0 1.0"/>
 </joint>
 <joint name="강체 4" type="fixed">
-  <origin xyz="0.0 -0.02 0.063" rpy="0 0 0"/>
+  <origin xyz="0.06 0.08 0.063" rpy="0 0 0"/>
   <parent link="base_link"/>
   <child link="cam_1"/>
